File: Schematics/_autosave-Refill_Dispensary.kicad_sch (KiCad schematic)
At the start: 28 parts, among them Q1 2N3905, Q2 2N3905, Q3 2N3905, SW1 SW_Push, SW2 SW_Push, SW3 SW_Push, U1 RP2040, U2 Screen, U3 Flash Memory, U5 OPAMP

Commit message: some updates
Parts:
- added D1, D2: DIODE, symbol pspice:DIODE
- added R1, R2: R, symbol Device:R
Connections:
- net +12V: now also R2.1
- net GND: now also R1.2
- new net: R1.1, R2.2
Other:
- note added: "Potentiometers on the UI"
Changed lines of the file:
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@@
+    (stroke (width 0) (type default) (color 0 0 0 0))
+  )
+  (wire (pts (xy 176.53 136.525) (xy 176.53 139.7))
     (stroke (width 0) (type default) (color 0 0 0 0))
   )
@@
     (stroke (width 0) (type default) (color 0 0 0 0))
   )
+  (wire (pts (xy 176.53 156.845) (xy 176.53 159.385))
+    (stroke (width 0) (type default) (color 0 0 0 0))
+  )
   (wire (pts (xy 53.34 81.28) (xy 63.5 81.28))
     (stroke (width 0) (type default) (color 0 0 0 0))
@@
     (stroke (width 0) (type default) (color 0 0 0 0))
   )
+  (wire (pts (xy 176.53 147.32) (xy 176.53 149.225))
+    (stroke (width 0) (type default) (color 0 0 0 0))
+  )
   (wire (pts (xy 218.44 76.2) (xy 254 76.2))
     (stroke (width 0) (type default) (color 0 0 0 0))
@@
   )
   (text "We need:\n1. Voltage transformer\n2. Power supply " (at -26.035 64.77 0)
+    (effects (font (size 1.27 1.27)) (justify left bottom))
+  )
+  (text "Potentiometers on the UI\n" (at 28.575 150.495 0)
     (effects (font (size 1.27 1.27)) (justify left bottom))
   )
@@
     (pin "2")
   )
+  (symbol (lib_id "Device:R") (at 176.53 153.035 0) (unit 1)
+    (in_bom yes) (on_board yes) (fields_autoplaced)
+    (property "Reference" "R1" (id 0) (at 179.07 151.7649 0)
+      (effects (font (size 1.27 1.27)) (justify left))
+    )
+    (property "Value" "R" (id 1) (at 179.07 154.3049 0)
+      (effects (font (size 1.27 1.27)) (justify left))
+    )
+    (property "Footprint" "" (id 2) (at 174.752 153.035 90)
+      (effects (font (size 1.27 1.27)) hide)
+    )
+    (property "Datasheet" "~" (id 3) (at 176.53 153.035 0)
+      (effects (font (size 1.27 1.27)) hide)
+    )
+    (pin "1")
+    (pin "2")
+  )
   (symbol (lib_id "pspice:DIODE") (at 273.05 54.61 90) (unit 1)
     (in_bom yes) (on_board yes) (fields_autoplaced)
@@
     (pin "3")
   )
+  (symbol (lib_id "pspice:DIODE") (at 190.5 141.605 180) (unit 1)
+    (in_bom yes) (on_board yes)
+    (property "Reference" "D1" (id 0) (at 190.5 133.35 0))
+    (property "Value" "DIODE" (id 1) (at 190.5 135.89 0))
+    (property "Footprint" "" (id 2) (at 190.5 141.605 0)
+      (effects (font (size 1.27 1.27)) hide)
+    )
+    (property "Datasheet" "~" (id 3) (at 190.5 141.605 0)
+      (effects (font (size 1.27 1.27)) hide)
+    )
+    (pin "1")
+    (pin "2")
+  )
   (symbol (lib_id "Connector_Generic:Conn_02x01") (at 218.44 55.88 90) (unit 1)
     (in_bom yes) (on_board yes) (fields_autoplaced)
@@
     (pin "2")
   )
+  (symbol (lib_id "pspice:DIODE") (at 206.375 140.97 180) (unit 1)
+    (in_bom yes) (on_board yes) (fields_autoplaced)
+    (property "Reference" "D2" (id 0) (at 206.375 133.35 0))
+    (property "Value" "DIODE" (id 1) (at 206.375 135.89 0))
+    (property "Footprint" "" (id 2) (at 206.375 140.97 0)
+      (effects (font (size 1.27 1.27)) hide)
+    )
+    (property "Datasheet" "~" (id 3) (at 206.375 140.97 0)
+      (effects (font (size 1.27 1.27)) hide)
+    )
+    (pin "1")
+    (pin "2")
+  )
   (symbol (lib_id "Transistor_BJT:2N3905") (at 175.26 40.64 0) (unit 1)
     (in_bom yes) (on_board yes) (fields_autoplaced)
@@
     (pin "1")
     (pin "2")
+  )
+  (symbol (lib_id "power:+12V") (at 176.53 136.525 0) (unit 1)
+    (in_bom yes) (on_board yes) (fields_autoplaced)
+    (property "Reference" "#PWR?" (id 0) (at 176.53 140.335 0)
+      (effects (font (size 1.27 1.27)) hide)
+    )
+    (property "Value" "+12V" (id 1) (at 176.53 130.81 0))
+    (property "Footprint" "" (id 2) (at 176.53 136.525 0)
+      (effects (font (size 1.27 1.27)) hide)
+    )
+    (property "Datasheet" "" (id 3) (at 176.53 136.525 0)
+      (effects (font (size 1.27 1.27)) hide)
+    )
+    (pin "1")
   )
   (symbol (lib_id "Device:LED") (at 57.15 38.1 90) (unit 1)
@@
     (pin "2")
   )
+  (symbol (lib_id "power:GND") (at 176.53 159.385 0) (unit 1)
+    (in_bom yes) (on_board yes) (fields_autoplaced)
+    (property "Reference" "#PWR?" (id 0) (at 176.53 165.735 0)
+      (effects (font (size 1.27 1.27)) hide)
+    )
+    (property "Value" "GND" (id 1) (at 176.53 163.83 0))
+    (property "Footprint" "" (id 2) (at 176.53 159.385 0)
+      (effects (font (size 1.27 1.27)) hide)
+    )
+    (property "Datasheet" "" (id 3) (at 176.53 159.385 0)
+      (effects (font (size 1.27 1.27)) hide)
+    )
+    (pin "1")
+  )
   (symbol (lib_id "power:+3.3V") (at 138.43 29.21 0) (unit 1)
     (in_bom yes) (on_board yes) (fields_autoplaced)
@@
     )
     (pin "1")
+  )
+  (symbol (lib_id "Device:R") (at 176.53 143.51 0) (unit 1)
+    (in_bom yes) (on_board yes) (fields_autoplaced)
+    (property "Reference" "R2" (id 0) (at 178.435 142.2399 0)
+      (effects (font (size 1.27 1.27)) (justify left))
+    )
+    (property "Value" "R" (id 1) (at 178.435 144.7799 0)
+      (effects (font (size 1.27 1.27)) (justify left))
+    )
+    (property "Footprint" "" (id 2) (at 174.752 143.51 90)
+      (effects (font (size 1.27 1.27)) hide)
+    )
+    (property "Datasheet" "~" (id 3) (at 176.53 143.51 0)
+      (effects (font (size 1.27 1.27)) hide)
+    )
+    (pin "1")
+    (pin "2")
   )
   (symbol (lib_id "Device:R") (at 247.65 128.27 180) (unit 1)
@@
       (reference "#PWR?") (unit 1) (value "GND") (footprint "")
     )
+    (path "/7b8fe0c7-fe6b-4683-9f56-6a49b76d106d"
+      (reference "#PWR?") (unit 1) (value "+12V") (footprint "")
+    )
     (path "/ad14d14d-5413-4a2e-86c0-956f71fb2a97"
       (reference "#PWR?") (unit 1) (value "GND") (footprint "")
@@
       (reference "#PWR?") (unit 1) (value "+3.3V") (footprint "")
     )
+    (path "/cb06d24d-772e-449d-8ee8-94749b85147e"
+      (reference "#PWR?") (unit 1) (value "GND") (footprint "")
+    )
     (path "/cc4cf2d1-80ff-4e15-859f-abe43d8868f4"
       (reference "#PWR?") (unit 1) (value "+3.3V") (footprint "")
@@
       (reference "C1") (unit 1) (value "100n") (footprint "")
     )
+    (path "/50f0d007-b0d2-42e8-8a0b-b3f00ff85096"
+      (reference "D1") (unit 1) (value "DIODE") (footprint "")
+    )
     (path "/ffe4d0fa-8210-4242-b4d8-6f2fa8ec1711"
       (reference "D1") (unit 1) (value "LED") (footprint "")
     )
+    (path "/61e04159-1cee-4a3f-aae1-d91a86514ce7"
+      (reference "D2") (unit 1) (value "DIODE") (footprint "")
+    )
     (path "/fd48bf1a-0220-4d04-a91b-d45f2f7592de"
       (reference "D2") (unit 1) (value "LED") (footprint "")
@@
       (reference "Q3") (unit 1) (value "2N3905") (footprint "Package_TO_SOT_THT:TO-92_Inline")
     )
+    (path "/21768582-a4a0-49d7-bc69-dfc1e28bd792"
+      (reference "R1") (unit 1) (value "R") (footprint "")
+    )
+    (path "/e838471f-7d7d-4ada-a948-aaabee10ea1c"
+      (reference "R2") (unit 1) (value "R") (footprint "")
+    )
     (path "/1e240b08-0d16-4025-99b5-bd51c48801a1"
