File: Schematics/Refill_Dispensary.kicad_sch (KiCad schematic)
At the start: 64 parts, among them J1 USB_B_Micro, J10 Switch 2, J11 Switch 3, J12 Switch 1, J2 Pot 1, J3 Barrel_Jack_Switch, J4 USB_BOOT, J5 Load Cell Power, J6 Load Cell Data, J7 Inductor 1, J8 Inductor 2, J9 Pot 2, Q1 TIP120, Q2 TIP120, SW4 SW_SPDT, U1 RP2040, U2 NCP1117-3.3_SOT223, U3 Flash Memory, U4 NHD-C0220BIZ, U5 AD622, Y1 Crystal

Commit message: board v1
Parts:
- added J13, J?: SWD, Connector_JST:JST_XH_B3B-XH-AM_1x03_P2.50mm_Vertical, symbol Connector_Generic:Conn_01x03
Connections:
- net +3.3V: now also J?.2 (Pin_2)
- net GND: now also J13.1 (Pin_1), J?.1 (Pin_1); no longer U5.5 (Ref)
- net SWCLK: now reaches U1.24 (SWCLK)
- net SWCLK: now also J13.2 (Pin_2)
- net SWD: now reaches U1.25 (SWD)
- net SWD: now also J13.3 (Pin_3)
- new net: J?.3 (Pin_3), U5.5 (Ref)
Changed lines of the file:
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@@
   (junction (at 240.03 71.12) (diameter 0) (color 0 0 0 0)
   )
-  (junction (at 335.28 110.49) (diameter 0) (color 0 0 0 0)
-  )
   (junction (at 31.75 251.46) (diameter 0) (color 0 0 0 0)
   )
@@
     (stroke (width 0) (type default) (color 0 0 0 0))
   )
+  (wire (pts (xy 187.96 167.64) (xy 194.31 167.64))
+    (stroke (width 0) (type default) (color 0 0 0 0))
+  )
   (wire (pts (xy 297.18 104.14) (xy 300.99 104.14))
     (stroke (width 0) (type default) (color 0 0 0 0))
@@
     (stroke (width 0) (type default) (color 0 0 0 0))
   )
+  (wire (pts (xy 340.36 110.49) (xy 340.36 120.65))
+    (stroke (width 0) (type default) (color 0 0 0 0))
+  )
   (wire (pts (xy 96.52 236.22) (xy 96.52 240.03))
     (stroke (width 0) (type default) (color 0 0 0 0))
@@
     (stroke (width 0) (type default) (color 0 0 0 0))
   )
+  (wire (pts (xy 187.96 170.18) (xy 194.31 170.18))
+    (stroke (width 0) (type default) (color 0 0 0 0))
+  )
   (wire (pts (xy 96.52 233.68) (xy 96.52 231.14))
     (stroke (width 0) (type default) (color 0 0 0 0))
@@
   )
   (wire (pts (xy 72.39 267.97) (xy 80.01 267.97))
-    (stroke (width 0) (type default) (color 0 0 0 0))
-  )
-  (wire (pts (xy 335.28 110.49) (xy 340.36 110.49))
     (stroke (width 0) (type default) (color 0 0 0 0))
   )
@@
     (effects (font (size 1.27 1.27)) (justify left bottom))
   )
+  (label "SWD" (at 187.96 170.18 0)
+    (effects (font (size 1.27 1.27)) (justify left bottom))
+  )
   (label "LED3" (at 44.45 234.95 0)
     (effects (font (size 1.27 1.27)) (justify left bottom))
@@
     (effects (font (size 1.27 1.27)) (justify left bottom))
   )
+  (label "SWCLK" (at 157.48 175.26 0)
+    (effects (font (size 1.27 1.27)) (justify left bottom))
+  )
+  (label "SWD" (at 157.48 172.72 0)
+    (effects (font (size 1.27 1.27)) (justify left bottom))
+  )
   (label "QSPI_SD0" (at 184.15 124.46 0)
     (effects (font (size 1.27 1.27)) (justify left bottom))
@@
   )
   (label "USB_D-" (at 168.91 111.76 0)
+    (effects (font (size 1.27 1.27)) (justify left bottom))
+  )
+  (label "SWCLK" (at 187.96 167.64 0)
     (effects (font (size 1.27 1.27)) (justify left bottom))
   )
@@
     (pin "2")
   )
+  (symbol (lib_id "Connector_Generic:Conn_01x03") (at 342.9 125.73 270) (unit 1)
+    (in_bom yes) (on_board yes) (fields_autoplaced)
+    (property "Reference" "J?" (id 0) (at 347.98 124.4599 90)
+      (effects (font (size 1.27 1.27)) (justify left))
+    )
+    (property "Value" "SWD" (id 1) (at 347.98 126.9999 90)
+      (effects (font (size 1.27 1.27)) (justify left))
+    )
+    (property "Footprint" "Connector_JST:JST_XH_B3B-XH-AM_1x03_P2.50mm_Vertical" (id 2) (at 342.9 125.73 0)
+      (effects (font (size 1.27 1.27)) hide)
+    )
+    (property "Datasheet" "~" (id 3) (at 342.9 125.73 0)
+      (effects (font (size 1.27 1.27)) hide)
+    )
+    (pin "1")
+    (pin "2")
+    (pin "3")
+  )
   (symbol (lib_id "Device:C") (at 248.92 67.31 180) (unit 1)
     (in_bom yes) (on_board yes) (fields_autoplaced)
@@
     )
   )
+  (symbol (lib_id "power:GND") (at 345.44 120.65 90) (unit 1)
+    (in_bom yes) (on_board yes) (fields_autoplaced)
+    (property "Reference" "#PWR?" (id 0) (at 351.79 120.65 0)
+      (effects (font (size 1.27 1.27)) hide)
+    )
+    (property "Value" "GND" (id 1) (at 349.25 120.6499 90)
+      (effects (font (size 1.27 1.27)) (justify right))
+    )
+    (property "Footprint" "" (id 2) (at 345.44 120.65 0)
+      (effects (font (size 1.27 1.27)) hide)
+    )
+    (property "Datasheet" "" (id 3) (at 345.44 120.65 0)
+      (effects (font (size 1.27 1.27)) hide)
+    )
+    (pin "1")
+  )
   (symbol (lib_id "Mechanical:MountingHole") (at 99.06 69.85 0) (unit 1)
     (in_bom yes) (on_board yes) (fields_autoplaced)
@@
       (effects (font (size 1.27 1.27)) hide)
     )
+  )
+  (symbol (lib_id "Connector_Generic:Conn_01x03") (at 152.4 175.26 180) (unit 1)
+    (in_bom yes) (on_board yes) (fields_autoplaced)
+    (property "Reference" "J13" (id 0) (at 152.4 166.37 0))
+    (property "Value" "SWD" (id 1) (at 152.4 168.91 0))
+    (property "Footprint" "Connector_JST:JST_XH_B3B-XH-AM_1x03_P2.50mm_Vertical" (id 2) (at 152.4 175.26 0)
+      (effects (font (size 1.27 1.27)) hide)
+    )
+    (property "Datasheet" "~" (id 3) (at 152.4 175.26 0)
+      (effects (font (size 1.27 1.27)) hide)
+    )
+    (pin "1")
+    (pin "2")
+    (pin "3")
   )
   (symbol (lib_id "Display_Character:NHD-C0220BIZ") (at 124.46 236.22 0) (unit 1)
@@
     (pin "1")
   )
+  (symbol (lib_id "power:GND") (at 157.48 177.8 0) (unit 1)
+    (in_bom yes) (on_board yes) (fields_autoplaced)
+    (property "Reference" "#PWR0139" (id 0) (at 157.48 184.15 0)
+      (effects (font (size 1.27 1.27)) hide)
+    )
+    (property "Value" "GND" (id 1) (at 157.48 182.88 0))
+    (property "Footprint" "" (id 2) (at 157.48 177.8 0)
+      (effects (font (size 1.27 1.27)) hide)
+    )
+    (property "Datasheet" "" (id 3) (at 157.48 177.8 0)
+      (effects (font (size 1.27 1.27)) hide)
+    )
+    (pin "1")
+  )
   (symbol (lib_id "power:+3.3V") (at 222.25 63.5 0) (unit 1)
     (in_bom yes) (on_board yes) (fields_autoplaced)
@@
     (pin "1")
     (pin "2")
+  )
+  (symbol (lib_id "power:+3.3V") (at 342.9 120.65 0) (unit 1)
+    (in_bom yes) (on_board yes) (fields_autoplaced)
+    (property "Reference" "#PWR?" (id 0) (at 342.9 124.46 0)
+      (effects (font (size 1.27 1.27)) hide)
+    )
+    (property "Value" "+3.3V" (id 1) (at 342.9 115.57 0))
+    (property "Footprint" "" (id 2) (at 342.9 120.65 0)
+      (effects (font (size 1.27 1.27)) hide)
+    )
+    (property "Datasheet" "" (id 3) (at 342.9 120.65 0)
+      (effects (font (size 1.27 1.27)) hide)
+    )
+    (pin "1")
   )
   (symbol (lib_id "power:+3.3V") (at 148.59 97.79 0) (unit 1)
@@
       (reference "#PWR0138") (unit 1) (value "+1.1V") (footprint "")
     )
+    (path "/cbedd1bd-cd03-4b07-8708-a77b954f25f0"
+      (reference "#PWR0139") (unit 1) (value "GND") (footprint "")
+    )
+    (path "/6e8d9245-e0ab-4498-a15b-8fb304c9e918"
+      (reference "#PWR?") (unit 1) (value "GND") (footprint "")
+    )
+    (path "/d85a6186-1fb9-400f-a4bf-bd2670303853"
+      (reference "#PWR?") (unit 1) (value "+3.3V") (footprint "")
+    )
     (path "/eb502b63-af1a-4319-bc15-3a83ac3a1265"
       (reference "C1") (unit 1) (value "100n") (footprint "Capacitor_SMD:C_0402_1005Metric")
@@
       (reference "J12") (unit 1) (value "Switch 1") (footprint "Connector_JST:JST_XH_B2B-XH-AM_1x02_P2.50mm_Vertical")
     )
+    (path "/898690fc-320a-464d-9710-35c57f5725dd"
+      (reference "J13") (unit 1) (value "SWD") (footprint "Connector_JST:JST_XH_B3B-XH-AM_1x03_P2.50mm_Vertical")
+    )
+    (path "/301407c9-703c-46e7-82dc-e0300c9d1f56"
+      (reference "J?") (unit 1) (value "SWD") (footprint "Connector_JST:JST_XH_B3B-XH-AM_1x03_P2.50mm_Vertical")
+    )
     (path "/c777b314-1500-42bb-9e4a-065e115b607d"
