File: Schematics/Refill_Dispensary.kicad_sch (KiCad schematic)
At the start: 66 parts, among them J1 USB_B_Micro, J10 Switch 2, J11 Switch 3, J12 Switch 1, J13 SWD, J2 Pot 1, J3 Barrel_Jack_Switch, J4 USB_BOOT, J5 Load Cell Power, J6 Load Cell Data, J7 Inductor 1, J8 Inductor 2, J9 Pot 2, Q1 TIP120, Q2 TIP120, SW4 SW_SPDT, U1 RP2040, U2 NCP1117-3.3_SOT223, U3 Flash Memory, U4 NHD-C0220BIZ, U5 AD622, Y1 Crystal

Commit message: board v1.1
Parts:
- gave numbers to parts that had none: 1
Changed lines of the file:
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@@
   (symbol (lib_id "Connector_Generic:Conn_01x03") (at 342.9 125.73 270) (unit 1)
     (in_bom yes) (on_board yes) (fields_autoplaced)
-    (property "Reference" "J?" (id 0) (at 347.98 124.4599 90)
+    (property "Reference" "J14" (id 0) (at 347.98 124.4599 90)
       (effects (font (size 1.27 1.27)) (justify left))
     )
@@
   (symbol (lib_id "power:GND") (at 345.44 120.65 90) (unit 1)
     (in_bom yes) (on_board yes) (fields_autoplaced)
-    (property "Reference" "#PWR?" (id 0) (at 351.79 120.65 0)
+    (property "Reference" "#PWR0141" (id 0) (at 351.79 120.65 0)
       (effects (font (size 1.27 1.27)) hide)
     )
@@
   (symbol (lib_id "power:+3.3V") (at 342.9 120.65 0) (unit 1)
     (in_bom yes) (on_board yes) (fields_autoplaced)
-    (property "Reference" "#PWR?" (id 0) (at 342.9 124.46 0)
+    (property "Reference" "#PWR0140" (id 0) (at 342.9 124.46 0)
       (effects (font (size 1.27 1.27)) hide)
     )
@@
       (reference "#PWR0139") (unit 1) (value "GND") (footprint "")
     )
+    (path "/d85a6186-1fb9-400f-a4bf-bd2670303853"
+      (reference "#PWR0140") (unit 1) (value "+3.3V") (footprint "")
+    )
     (path "/6e8d9245-e0ab-4498-a15b-8fb304c9e918"
-      (reference "#PWR?") (unit 1) (value "GND") (footprint "")
-    )
-    (path "/d85a6186-1fb9-400f-a4bf-bd2670303853"
-      (reference "#PWR?") (unit 1) (value "+3.3V") (footprint "")
+      (reference "#PWR0141") (unit 1) (value "GND") (footprint "")
     )
     (path "/eb502b63-af1a-4319-bc15-3a83ac3a1265"
@@
     )
     (path "/301407c9-703c-46e7-82dc-e0300c9d1f56"
-      (reference "J?") (unit 1) (value "SWD") (footprint "Connector_JST:JST_XH_B3B-XH-AM_1x03_P2.50mm_Vertical")
+      (reference "J14") (unit 1) (value "SWD") (footprint "Connector_JST:JST_XH_B3B-XH-AM_1x03_P2.50mm_Vertical")
     )
     (path "/c777b314-1500-42bb-9e4a-065e115b607d"
